Commit message: changed robot model to sphere, added a small house world model that doesnt work in gazebo.

File: ros2_ws/src/ball_e_description/urdf/ball_e.urdf.xacro (robot description, xacro)
@@ -7,10 +7,10 @@
   <!-- Base footprint (reference frame on the ground) -->
   <link name="base_footprint"/>
-  <!-- Base link (main body) -->
+  <!-- Base link (main body) - Ball shaped -->
   <link name="base_link">
     <visual>
-      <origin xyz="0 0 0.05" rpy="0 0 0"/>
+      <origin xyz="0 0 0.1" rpy="0 0 0"/>
       <geometry>
-        <cylinder radius="0.15" length="0.1"/>
+        <sphere radius="0.1"/>
       </geometry>
       <material name="blue">
@@ -19,15 +19,16 @@
     </visual>
     <collision>
-      <origin xyz="0 0 0.05" rpy="0 0 0"/>
+      <origin xyz="0 0 0.1" rpy="0 0 0"/>
       <geometry>
-        <cylinder radius="0.15" length="0.1"/>
+        <sphere radius="0.1"/>
       </geometry>
     </collision>
     <inertial>
-      <origin xyz="0 0 0.05" rpy="0 0 0"/>
+      <origin xyz="0 0 0.1" rpy="0 0 0"/>
       <mass value="2.0"/>
-      <inertia ixx="0.00625" ixy="0.0" ixz="0.0"
-               iyy="0.00625" iyz="0.0"
-               izz="0.01125"/>
+      <!-- Inertia for solid sphere: I = 2/5 * m * r^2 = 2/5 * 2.0 * 0.1^2 = 0.004 -->
+      <inertia ixx="0.004" ixy="0.0" ixz="0.0"
+               iyy="0.004" iyz="0.0"
+               izz="0.004"/>
     </inertial>
   </link>
@@ -37,39 +38,9 @@
     <origin xyz="0 0 0" rpy="0 0 0"/>
   </joint>
-  <!-- Camera tower/mount -->
-  <link name="camera_mount">
-    <visual>
-      <origin xyz="0 0 0.075" rpy="0 0 0"/>
-      <geometry>
-        <box size="0.05 0.05 0.15"/>
-      </geometry>
-      <material name="dark_grey">
-        <color rgba="0.3 0.3 0.3 1.0"/>
-      </material>
-    </visual>
-    <collision>
-      <origin xyz="0 0 0.075" rpy="0 0 0"/>
-      <geometry>
-        <box size="0.05 0.05 0.15"/>
-      </geometry>
-    </collision>
-    <inertial>
-      <origin xyz="0 0 0.075" rpy="0 0 0"/>
-      <mass value="0.2"/>
-      <inertia ixx="0.0004" ixy="0.0" ixz="0.0"
-               iyy="0.0004" iyz="0.0"
-               izz="0.00005"/>
-    </inertial>
-  </link>
-  <joint name="camera_mount_joint" type="fixed">
-    <parent link="base_link"/>
-    <child link="camera_mount"/>
-    <origin xyz="0 0 0.1" rpy="0 0 0"/>
-  </joint>
-  <!-- Instantiate camera sensor -->
+  <!-- Instantiate camera sensor - integrated in top hemisphere -->
   <xacro:camera_sensor
-    parent="camera_mount"
+    parent="base_link"
     name="camera"
-    xyz="0 0 0.15"
+    xyz="0.05 0 0.18"
     rpy="0 0 0"/>
   <!-- Wheels (visual only for now, will add control later) -->
@@ -101,5 +72,5 @@
     <parent link="base_link"/>
     <child link="left_wheel"/>
-    <origin xyz="0 0.08 0.033" rpy="0 0 0"/>
+    <origin xyz="0 0.09 0.1" rpy="0 0 0"/>
     <axis xyz="0 1 0"/>
   </joint>
@@ -131,5 +102,5 @@
     <parent link="base_link"/>
     <child link="right_wheel"/>
-    <origin xyz="0 -0.08 0.033" rpy="0 0 0"/>
+    <origin xyz="0 -0.09 0.1" rpy="0 0 0"/>
     <axis xyz="0 1 0"/>
   </joint>
@@ -162,5 +133,5 @@
     <parent link="base_link"/>
     <child link="caster_wheel"/>
-    <origin xyz="-0.1 0 0.01" rpy="0 0 0"/>
+    <origin xyz="-0.07 0 0.02" rpy="0 0 0"/>
   </joint>
   <!-- Gazebo Classic Differential Drive Plugin -->
@@ -176,5 +147,5 @@
       <right_joint>right_wheel_joint</right_joint>
       <!-- Kinematics -->
-      <wheel_separation>0.16</wheel_separation>
+      <wheel_separation>0.18</wheel_separation>
       <wheel_diameter>0.066</wheel_diameter>
       <!-- Limits -->

File: ros2_ws/src/ball_e_description/urdf/camera.xacro (robot description, xacro)
@@ -2,10 +2,10 @@
 <robot xmlns:xacro="http://www.ros.org/wiki/xacro">
   <xacro:macro name="camera_sensor" params="parent name xyz rpy">
-    <!-- Camera link -->
+    <!-- Camera link - small cylindrical protrusion -->
     <link name="${name}_link">
       <visual>
-        <origin xyz="0 0 0" rpy="0 0 0"/>
+        <origin xyz="0.005 0 0" rpy="0 1.5708 0"/>
         <geometry>
-          <box size="0.02 0.05 0.02"/>
+          <cylinder radius="0.015" length="0.01"/>
         </geometry>
         <material name="camera_grey">
@@ -14,7 +14,7 @@
       </visual>
       <collision>
-        <origin xyz="0 0 0" rpy="0 0 0"/>
+        <origin xyz="0.005 0 0" rpy="0 1.5708 0"/>
         <geometry>
-          <box size="0.02 0.05 0.02"/>
+          <cylinder radius="0.015" length="0.01"/>
         </geometry>
       </collision>
